File: Break out board/round_2/_saved_round_2.sch (KiCad schematic (older format))
At the start: 2 parts, among them U1 LSM90S1

Commit message: Did everything
Parts:
- added D1, D2: D, Diode_SMD:D_0603_1608Metric_Pad1.05x0.95mm_HandSolder, symbol Device:D
- added R1, R3: 0, Resistor_SMD:R_0603_1608Metric_Pad1.05x0.95mm_HandSolder, symbol Device:R
- added R2, R4: 1K, Resistor_SMD:R_0603_1608Metric_Pad1.05x0.95mm_HandSolder, symbol Device:R
- added R5, R6: 500, Resistor_SMD:R_0603_1608Metric_Pad1.05x0.95mm_HandSolder, symbol Device:R
Connections:
- net labels added: +3V3, DRDYM, GND, INT1AG, INT2AG, INTM, SCL, SDA, SDOAG, SDOM
- wire segments 42 -> 6
