File: Break out board/round_2/round_2.sch (KiCad schematic (older format))
At the start: 2 parts, among them U1 LSM90S1

Commit message: Did everything
Parts:
- added R1, R3: 0, Resistor_SMD:R_0603_1608Metric_Pad1.05x0.95mm_HandSolder, symbol Device:R
- added R2, R4: 1K, Resistor_SMD:R_0603_1608Metric_Pad1.05x0.95mm_HandSolder, symbol Device:R
Connections:
- net labels added: +3V3, DRDYM, GND, INT1AG, INT2AG, INTM, SCL, SDA, SDOAG, SDOM
- wire segments 42 -> 4
Changed lines of the file:
@@
 EESchema Schematic File Version 4
+LIBS:round_2-cache
 EELAYER 26 0
 EELAYER END
@@
 L MRDT_Sensors:LSM90S1 U1
 U 1 1 5BBD7441
-P 5200 4100
-F 0 "U1" H 5250 4050 60  0001 C CNN
-F 1 "LSM90S1" H 5550 4891 60  0000 C CNN
-F 2 "MRDT_Sensors:IMU_LSM90S1" H 5250 4100 60  0001 C CNN
-F 3 "" H 5250 4100 60  0001 C CNN
-	1    5200 4100
+P 4200 2950
+F 0 "U1" H 4250 2900 60  0001 C CNN
+F 1 "LSM90S1" H 4550 3741 60  0000 C CNN
+F 2 "MRDT_Sensors:IMU_LSM90S1" H 4250 2950 60  0001 C CNN
+F 3 "" H 4250 2950 60  0001 C CNN
+	1    4200 2950
 	1    0    0    -1
 $EndComp
@@
 L MRDT_Connectors:Molex_SL_08 Conn1
 U 1 1 5BBD7471
-P 5150 4900
-F 0 "Conn1" V 5040 5738 60  0000 L CNN
-F 1 "Molex_SL_08" V 5146 5738 60  0000 L CNN
-F 2 "MRDT_Connectors:MOLEX_SL_08_Horizontal" H 5150 5200 60  0001 C CNN
-F 3 "" H 5150 5200 60  0001 C CNN
-	1    5150 4900
+P 6350 3100
+F 0 "Conn1" V 6240 3938 60  0000 L CNN
+F 1 "Molex_SL_08" V 6346 3938 60  0000 L CNN
+F 2 "MRDT_Connectors:MOLEX_SL_08_Horizontal" H 6350 3400 60  0001 C CNN
+F 3 "" H 6350 3400 60  0001 C CNN
+	1    6350 3100
+	1    0    0    -1
+$EndComp
+Text GLabel 4000 2300 0    50   Input ~ 0
++3V3
+Text GLabel 5100 2350 2    50   UnSpc ~ 0
+GND
+Text GLabel 4000 2800 0    50   Input ~ 0
++3V3
+Text GLabel 5100 2450 2    50   Input ~ 0
++3V3
+Text GLabel 6150 3050 0    50   Input ~ 0
++3V3
+Text GLabel 4000 2900 0    50   Input ~ 0
++3V3
+Text GLabel 6150 2350 0    50   UnSpc ~ 0
+GND
+Text GLabel 6150 2450 0    50   Input ~ 0
+INT2AG
+Text GLabel 6150 2550 0    50   Input ~ 0
+INT1AG
+Text GLabel 6150 2650 0    50   Input ~ 0
+INTM
+Text GLabel 6150 2750 0    50   Input ~ 0
+DRDYM
+Text GLabel 6150 2850 0    50   Input ~ 0
+SDA
+Text GLabel 6150 2950 0    50   Input ~ 0
+SCL
+Text GLabel 4000 2500 0    50   Output ~ 0
+SDA
+Text GLabel 4000 2400 0    50   Output ~ 0
+SCL
+Text GLabel 5100 2550 2    50   Output ~ 0
+INT2AG
+Text GLabel 5100 2650 2    50   Output ~ 0
+INT1AG
+Text GLabel 5100 2750 2    50   Output ~ 0
+INTM
+Text GLabel 5100 2850 2    50   Output ~ 0
+DRDYM
+Text GLabel 3050 3550 0    50   Input ~ 0
++3V3
+Text GLabel 4550 3550 0    50   Input ~ 0
++3V3
+Text GLabel 3450 3850 3    50   UnSpc ~ 0
+GND
+Text GLabel 5000 3850 3    50   UnSpc ~ 0
+GND
+$Comp
+L Device:R R2
+U 1 1 5BCD1016
+P 3450 3700
+F 0 "R2" H 3520 3746 50  0000 L CNN
+F 1 "1K" H 3520 3655 50  0000 L CNN
+F 2 "Resistor_SMD:R_0603_1608Metric_Pad1.05x0.95mm_HandSolder" V 3380 3700 50  0001 C CNN
+F 3 "~" H 3450 3700 50  0001 C CNN
+	1    3450 3700
+	1    0    0    -1
+$EndComp
+$Comp
+L Device:R R4
+U 1 1 5BCD1060
+P 5000 3700
+F 0 "R4" H 5070 3746 50  0000 L CNN
+F 1 "1K" H 5070 3655 50  0000 L CNN
+F 2 "Resistor_SMD:R_0603_1608Metric_Pad1.05x0.95mm_HandSolder" V 4930 3700 50  0001 C CNN
+F 3 "~" H 5000 3700 50  0001 C CNN
+	1    5000 3700
+	1    0    0    -1
+$EndComp
+$Comp
+L Device:R R1
+U 1 1 5BCD10FD
+P 3200 3550
+F 0 "R1" V 2993 3550 50  0000 C CNN
+F 1 "0" V 3084 3550 50  0000 C CNN
+F 2 "Resistor_SMD:R_0603_1608Metric_Pad1.05x0.95mm_HandSolder" V 3130 3550 50  0001 C CNN
+F 3 "~" H 3200 3550 50  0001 C CNN
+	1    3200 3550
+	0    1    1    0
+$EndComp
+$Comp
+L Device:R R3
+U 1 1 5BCD1148
+P 4700 3550
+F 0 "R3" V 4493 3550 50  0000 C CNN
+F 1 "0" V 4584 3550 50  0000 C CNN
+F 2 "Resistor_SMD:R_0603_1608Metric_Pad1.05x0.95mm_HandSolder" V 4630 3550 50  0001 C CNN
+F 3 "~" H 4700 3550 50  0001 C CNN
+	1    4700 3550
 	0    1    1    0
 $EndComp
 Wire Wire Line
-	5000 3450 4800 3450
+	3350 3550 3450 3550
 Wire Wire Line
-	4800 3450 4800 3750
+	4850 3550 5000 3550
+Connection ~ 5000 3550
 Wire Wire Line
-	4800 4700 5200 4700
+	5000 3550 5100 3550
+Connection ~ 3450 3550
 Wire Wire Line
-	5000 3750 4800 3750
-Connection ~ 4800 3750
-Wire Wire Line
-	4800 3750 4800 3850
-Wire Wire Line
-	5000 3850 4800 3850
-Connection ~ 4800 3850
-Wire Wire Line
-	4800 3850 4800 3950
-Wire Wire Line
-	5200 4700 5200 4150
-Wire Wire Line
-	5200 4150 6250 4150
-Wire Wire Line
-	6250 4150 6250 3600
-Wire Wire Line
-	6250 3600 6100 3600
-Connection ~ 5200 4700
-Wire Wire Line
-	5000 4050 4800 4050
-Connection ~ 4800 4050
-Wire Wire Line
-	4800 4050 4800 4700
-Wire Wire Line
-	5000 3950 4800 3950
-Connection ~ 4800 3950
-Wire Wire Line
-	4800 3950 4800 4050
-Wire Wire Line
-	5000 3550 4850 3550
-Wire Wire Line
-	4850 3550 4850 4500
-Wire Wire Line
-	4850 4500 5300 4500
-Wire Wire Line
-	5300 4500 5300 4700
-Wire Wire Line
-	5000 3650 4900 3650
-Wire Wire Line
-	4900 3650 4900 4450
-Wire Wire Line
-	4900 4450 5400 4450
-Wire Wire Line
-	5400 4450 5400 4700
-Wire Wire Line
-	6100 4000 6100 4450
-Wire Wire Line
-	6100 4450 5500 4450
-Wire Wire Line
-	5500 4450 5500 4700
-Wire Wire Line
-	6100 3900 6150 3900
-Wire Wire Line
-	6150 3900 6150 4500
-Wire Wire Line
-	6150 4500 5600 4500
-Wire Wire Line
-	5600 4500 5600 4700
-Wire Wire Line
-	6100 3800 6200 3800
-Wire Wire Line
-	6200 3800 6200 4550
-Wire Wire Line
-	6200 4550 5700 4550
-Wire Wire Line
-	5700 4550 5700 4700
-Wire Wire Line
-	6100 3700 6300 3700
-Wire Wire Line
-	6300 3700 6300 4600
-Wire Wire Line
-	6300 4600 5800 4600
-Wire Wire Line
-	5800 4600 5800 4700
-Wire Wire Line
-	6100 3500 6350 3500
-Wire Wire Line
-	6350 3500 6350 4650
-Wire Wire Line
-	6350 4650 5900 4650
-Wire Wire Line
-	5900 4650 5900 4700
+	3450 3550 3600 3550
+Text GLabel 3600 3550 2    50   Output ~ 0
+SDOAG
+Text GLabel 4000 2600 0    50   Input ~ 0
+SDOAG
+Text GLabel 4000 2700 0    50   Input ~ 0
+SDOM
+Text GLabel 5100 3550 2    50   Output ~ 0
+SDOM
 $EndSCHEMATC
