File: LSM9DS1Breakout_Hardware/LSM9DS1Breakout_Hardware.sch (KiCad schematic (older format))
At the start: 8 parts, among them U1 Adafruit_LSM9DS1

Commit message: created nano interface scheamtic
Parts:
- removed D1: LED, LED_SMD:LED_0603_1608Metric_Pad1.05x0.95mm_HandSolder, symbol Device:LED
- removed R1: 500, Resistor_SMD:R_0603_1608Metric_Pad1.05x0.95mm_HandSolder, symbol Device:R
Changed lines of the file:
@@
 Text Notes 4400 4450 0    50   ~ 0
-Yelo
-$Comp
-L Device:R R1
-U 1 1 5CB6CFCD
-P 3900 3950
-F 0 "R1" H 3970 3996 50  0000 L CNN
-F 1 "500" H 3970 3905 50  0000 L CNN
-F 2 "Resistor_SMD:R_0603_1608Metric_Pad1.05x0.95mm_HandSolder" V 3830 3950 50  0001 C CNN
-F 3 "~" H 3900 3950 50  0001 C CNN
-	1    3900 3950
-	1    0    0    -1
-$EndComp
-$Comp
-L Device:LED D1
-U 1 1 5CB6CFD3
-P 3900 4300
-F 0 "D1" V 3938 4183 50  0000 R CNN
-F 1 "LED" V 3847 4183 50  0000 R CNN
-F 2 "LED_SMD:LED_0603_1608Metric_Pad1.05x0.95mm_HandSolder" H 3900 4300 50  0001 C CNN
-F 3 "~" H 3900 4300 50  0001 C CNN
-	1    3900 4300
-	0    -1   -1   0
-$EndComp
-$Comp
-L power:GND #PWR0108
-U 1 1 5CB6CFDF
-P 3900 4500
-F 0 "#PWR0108" H 3900 4250 50  0001 C CNN
-F 1 "GND" H 3905 4327 50  0000 C CNN
-F 2 "" H 3900 4500 50  0001 C CNN
-F 3 "" H 3900 4500 50  0001 C CNN
-	1    3900 4500
-	1    0    0    -1
-$EndComp
-Wire Wire Line
-	3900 3750 3900 3800
-Wire Wire Line
-	3900 4100 3900 4150
-Wire Wire Line
-	3900 4450 3900 4500
-Text Notes 4000 4450 0    50   ~ 0
 Yelo
 Text GLabel 4300 3750 1    50   Input ~ 0
 SCL
-Text GLabel 3900 3750 1    50   BiDi ~ 0
-SDA
 $EndSCHEMATC
