File: ArduinoNanoInterface_Hardware/ArduinoNanoInterface_Hardware.kicad_pcb (KiCad board)
At the start: 2 copper layers, 20.3 x 81.3 mm, 17 parts, among them Q1 BSS138, Q2 BSS138

Commit message: created gerbs
Parts:
- moved R3 9.85 mm to (95.5, 115.5)
- moved R4 7.73 mm to (91.4, 115.5)
- moved R2 3.66 mm to (89.7, 123.7), turned to 0 degrees
- moved R1 3.21 mm to (98.8, 123.7), turned to 0 degrees
- moved Q2 2.87 mm to (89.7, 121.2), turned to 90 degrees
- moved Q1 2.27 mm to (98.8, 121.2), turned to 90 degrees
Connections:
- Q1 pad 2: NanoTx -> Tx
- Q1 pad 3: Tx -> NanoTx
- Q2 pad 2: NanoRx -> Rx
- Q2 pad 3: Rx -> NanoRx
- R1 pad 2: NanoTx -> Tx
- R2 pad 2: NanoRx -> Rx
- R3 pad 2: Tx -> NanoTx
- R4 pad 2: Rx -> NanoRx
Routing:
- net +3V3: track 26.7 -> 39.1 mm
- net NanoTx: track 25.6 -> 28.4 mm
- net NanoRx: track 33.1 -> 30.7 mm
- net +5V: track 11.2 -> 13.1 mm, vias 1 -> 2
- net Rx: track 15.2 -> 13.7 mm
- net Tx: track 16.4 -> 15.8 mm
