File: ArduinoNanoInterface_Hardware/ArduinoNanoInterface_Hardware.sch (KiCad schematic (older format))
At the start: 17 parts, among them Q1 BSS138, Q2 BSS138

Commit message: layout
Parts:
- JP1, JP2: footprint Connector_PinSocket_2.54mm:PinSocket_1x03_P2.54mm_Horizontal -> Connector_PinSocket_2.54mm:PinSocket_1x03_P2.54mm_Vertical
Connections:
- net HW_Rx: now also JP1.1; no longer JP1.3
- net SW_Rx: now also JP1.3; no longer JP1.1
Changed lines of the file:
@@
 F 0 "JP2" V 7454 2301 50  0000 L CNN
 F 1 "Jumper_NC_Dual" V 7300 1500 50  0000 L CNN
-F 2 "Connector_PinSocket_2.54mm:PinSocket_1x03_P2.54mm_Horizontal" H 7500 2200 50  0001 C CNN
+F 2 "Connector_PinSocket_2.54mm:PinSocket_1x03_P2.54mm_Vertical" H 7500 2200 50  0001 C CNN
 F 3 "~" H 7500 2200 50  0001 C CNN
 	1    7500 2200
@@
 F 0 "JP1" V 7454 1501 50  0000 L CNN
 F 1 "Jumper_NC_Dual" V 7300 700 50  0000 L CNN
-F 2 "Connector_PinSocket_2.54mm:PinSocket_1x03_P2.54mm_Horizontal" H 7500 1400 50  0001 C CNN
+F 2 "Connector_PinSocket_2.54mm:PinSocket_1x03_P2.54mm_Vertical" H 7500 1400 50  0001 C CNN
 F 3 "~" H 7500 1400 50  0001 C CNN
 	1    7500 1400
@@
 Wire Wire Line
 	5350 3500 5400 3500
+Text GLabel 7550 1100 2    50   Output ~ 0
+HW_Rx
 Text GLabel 7550 1700 2    50   Output ~ 0
-HW_Rx
-Text GLabel 7550 1100 2    50   Output ~ 0
 SW_Rx
 Text GLabel 7550 1900 2    50   Input ~ 0

Commit message: created gerbs
Connections:
- net NanoRx: now also Q2.3 (D), R4.2; no longer Q2.2 (S), R2.2
- net NanoTx: now also Q1.3 (D), R3.2; no longer Q1.2 (S), R1.2
- net Rx: now also Q2.2 (S), R2.2; no longer Q2.3 (D), R4.2
- net Tx: now also Q1.2 (S), R1.2; no longer Q1.3 (D), R3.2
Changed lines of the file:
@@
 EESchema Schematic File Version 4
+LIBS:ArduinoNanoInterface_Hardware-cache
 EELAYER 26 0
 EELAYER END
@@
 	1    0    0    -1
 $EndComp
-Text GLabel 3150 4200 0    50   Input ~ 0
+Text GLabel 3750 4200 2    50   Input ~ 0
 NanoTx
-Text GLabel 3750 4200 2    50   Output ~ 0
+Text GLabel 3150 4200 0    50   Output ~ 0
 Tx
 Wire Wire Line
@@
 Wire Wire Line
 	7500 2450 7500 2500
-Text Notes 10000 4500 0    50   ~ 0
-Green
 $Comp
 L Device:LED D3
@@
 	1    0    0    -1
 $EndComp
+Text GLabel 3750 5250 2    50   Output ~ 0
+NanoRx
 Text GLabel 3150 5250 0    50   Input ~ 0
-NanoRx
-Text GLabel 3750 5250 2    50   Output ~ 0
 Rx
 Wire Wire Line
